File: MCD.kicad_pcb (KiCad board)
At the start: 2 copper layers, 143.6 x 54.9 mm, 75 parts, among them J1 JTAG, J2 TTL, J3 5V JMP, SW1 RESET BTN, U1 RAM_LOW, U10 I2C_DATA, U11 IOIOI SHIFT, U12 I2C SHIFT, U13 SEEED XIAO ESP32C3, U14 3.69MHZ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

Commit message: Rev 1.1
Added pictures of PCB and readme
Parts:
- J3: value 5V JMP -> 5V
- moved G*** 0.95 mm to (212.8, 96.7)
Changed lines of the file:
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@@
         (effects (font (size 1 1) (thickness 0.15)))
     )
-    (fp_text value "5V JMP" (at 0 5.1) (layer "F.SilkS")
+    (fp_text value "5V" (at 0 5.1) (layer "F.SilkS")
         (effects (font (size 1 1) (thickness 0.15)))
     )
@@
   )
   (footprint "LOGO" (layer "F.Cu")
-    (at 211.9 96.4)
+    (at 212.8 96.7)
     (attr board_only exclude_from_pos_files exclude_from_bom)
     (fp_text reference "G***" (at 0 0) (layer "F.SilkS") hide
@@
     )
   )
-  (gr_line (start 220.4 106.7) (end 210.8 106.7)
+  (gr_line (start 221.3 107) (end 211.7 107)
     (stroke (width 0.15) (type default)) (layer "F.SilkS"))
   (gr_line (start 112.6 97.3) (end 112.6 103.7)
@@
   (gr_line (start 221.5 124.1) (end 222 124.1)
     (stroke (width 0.15) (type default)) (layer "F.SilkS"))
-  (gr_line (start 207.6 106.7) (end 210.1 106.7)
+  (gr_line (start 208.5 107) (end 211 107)
     (stroke (width 0.15) (type default)) (layer "F.SilkS"))
   (gr_line (start 135.7 134.8) (end 175.6 134.8)
@@
     )
   )
-  (gr_text "jaedynchilton.com" (at 207.1 106) (layer "F.SilkS")
+  (gr_text "jaedynchilton.com" (at 208 106.3) (layer "F.SilkS")
     (effects (font (size 1 1) (thickness 0.15)) (justify left))
   )
@@
     )
   )
+  (group "" (id e27361d7-3e7b-4c88-9095-c8e83b50eae9)
+    (members
+      0a3631ca-98d9-452f-a3d2-d78f1c713965
+      6bb49f1c-1f28-444b-b88b-f281d6525c9f
+      82840cd3-8980-4524-8249-2a8671282db3
+      837088b7-6563-4fdc-97aa-c5e78932e090
+    )
+  )
