File: MCD.kicad_sch (KiCad schematic)
At the start: 61 parts, among them J1 JTAG, J2 TTL, J3 5V JMP, SW1 RESET BTN, U1 RAM_LOW, U10 I2C_DATA, U11 IOIOI SHIFT, U12 I2C SHIFT, U13 SEEED XIAO ESP32C3, U14 3.69MHZ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

Commit message: Rev 1.1
Added pictures of PCB and readme
Parts:
- J3: value 5V JMP -> 5V
Changed lines of the file:
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@@
       (effects (font (size 1.27 1.27)) (justify left))
     )
-    (property "Value" "5V JMP" (at 292.1 192.405 0)
+    (property "Value" "5V" (at 292.1 192.405 0)
       (effects (font (size 1.27 1.27)) (justify left))
     )
